Commit message: Install meshes of robot UR5
  - install in package hpp_practicals to avoid conflict with ur_description,
    modify urdf accordingly.

File: urdf/ur5_joint_limited_robot.urdf (robot description, URDF)
Before this commit: robot ur5, 11 links, 10 joints
Links:
- link base_link: geometry collision mesh filename=package://hpp_practicals/meshes/ur5/collision/base.stl; visual mesh filename=package://hpp_practicals/meshes/ur5/visual/base.osg
- link forearm_link: geometry collision mesh filename=package://hpp_practicals/meshes/ur5/collision/forearm.stl; visual mesh filename=package://hpp_practicals/meshes/ur5/visual/forearm.osg
- link shoulder_link: geometry collision mesh filename=package://hpp_practicals/meshes/ur5/collision/shoulder.stl; visual mesh filename=package://hpp_practicals/meshes/ur5/visual/shoulder.osg
- link upper_arm_link: geometry collision mesh filename=package://hpp_practicals/meshes/ur5/collision/upperarm.stl; visual mesh filename=package://hpp_practicals/meshes/ur5/visual/upperarm.osg
- link wrist_1_link: geometry collision mesh filename=package://hpp_practicals/meshes/ur5/collision/wrist1.stl; visual mesh filename=package://hpp_practicals/meshes/ur5/visual/wrist1.osg
- link wrist_2_link: geometry collision mesh filename=package://hpp_practicals/meshes/ur5/collision/wrist2.stl; visual mesh filename=package://hpp_practicals/meshes/ur5/visual/wrist2.osg
- link wrist_3_link: geometry collision mesh filename=package://hpp_practicals/meshes/ur5/collision/wrist3.stl; visual mesh filename=package://hpp_practicals/meshes/ur5/visual/wrist3.osg
